File: kicad/hdmi-csi.kicad_sch (KiCad schematic)
At the start: 6 parts, among them CN1 10029449-111RLF

Commit message: Replace files.
Parts:
- added J1: USB_C_Receptacle, symbol Connector:USB_C_Receptacle
- added J2: USB_C_Receptacle_PowerOnly_6P, symbol Connector:USB_C_Receptacle_PowerOnly_6P
Connections:
- new net: J1.A1 (GND), J1.A12 (GND), J1.B1 (GND), J1.B12 (GND)
- new net: J1.A4 (VBUS), J1.A9 (VBUS), J1.B4 (VBUS), J1.B9 (VBUS)
- new net: J2.A12 (GND), J2.B12 (GND)
- new net: J2.A9 (VBUS), J2.B9 (VBUS)
Changed lines of the file:
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@@
+	)
+	(symbol
+		(lib_id "Connector:USB_C_Receptacle")
+		(at 35.56 59.69 0)
+		(unit 1)
+		(exclude_from_sim no)
+		(in_bom yes)
+		(on_board yes)
+		(dnp no)
+		(fields_autoplaced yes)
+		(property "Reference" "J1"
+			(at 35.56 26.67 0)
+			(effects
+				(font
+					(size 1.27 1.27)
+				)
+			)
+		)
+		(property "Value" "USB_C_Receptacle"
+			(at 35.56 29.21 0)
+			(effects
+				(font
+					(size 1.27 1.27)
+				)
+			)
+		)
+		(property "Footprint" ""
+			(at 39.37 59.69 0)
+			(effects
+				(font
+					(size 1.27 1.27)
+				)
+				(hide yes)
+			)
+		)
+		(property "Datasheet" "https://www.usb.org/sites/default/files/documents/usb_type-c.zip"
+			(at 39.37 59.69 0)
+			(effects
+				(font
+					(size 1.27 1.27)
+				)
+				(hide yes)
+			)
+		)
+		(property "Description" "USB Full-Featured Type-C Receptacle connector"
+			(at 35.56 59.69 0)
+			(effects
+				(font
+					(size 1.27 1.27)
+				)
+				(hide yes)
+			)
+		)
+		(pin "A6"
+		)
+		(pin "B3"
+		)
+		(pin "B9"
+		)
+		(pin "A7"
+		)
+		(pin "B4"
+		)
+		(pin "A1"
+		)
+		(pin "B10"
+		)
+		(pin "A12"
+		)
+		(pin "A8"
+		)
+		(pin "A11"
+		)
+		(pin "S1"
+		)
+		(pin "B12"
+		)
+		(pin "B7"
+		)
+		(pin "A4"
+		)
+		(pin "A5"
+		)
+		(pin "B6"
+		)
+		(pin "B8"
+		)
+		(pin "A2"
+		)
+		(pin "A10"
+		)
+		(pin "A9"
+		)
+		(pin "B5"
+		)
+		(pin "B1"
+		)
+		(pin "B2"
+		)
+		(pin "B11"
+		)
+		(pin "A3"
+		)
+		(instances
+			(project ""
+				(path "/804d8951-ccf0-42ec-be9a-378a7536c3df"
+					(reference "J1")
+					(unit 1)
+				)
+			)
+		)
 	)
 	(symbol
@@
 					(unit 1)
 				)
+			)
+		)
+	)
+	(symbol
+		(lib_id "Connector:USB_C_Receptacle_PowerOnly_6P")
+		(at 74.93 44.45 0)
+		(unit 1)
+		(exclude_from_sim no)
+		(in_bom yes)
+		(on_board yes)
+		(dnp no)
+		(fields_autoplaced yes)
+		(property "Reference" "J2"
+			(at 74.93 26.67 0)
+			(effects
+				(font
+					(size 1.27 1.27)
+				)
+			)
+		)
+		(property "Value" "USB_C_Receptacle_PowerOnly_6P"
+			(at 74.93 29.21 0)
+			(effects
+				(font
+					(size 1.27 1.27)
+				)
+			)
+		)
+		(property "Footprint" ""
+			(at 78.74 41.91 0)
+			(effects
+				(font
+					(size 1.27 1.27)
+				)
+				(hide yes)
+			)
+		)
+		(property "Datasheet" "https://www.usb.org/sites/default/files/documents/usb_type-c.zip"
+			(at 74.93 44.45 0)
+			(effects
+				(font
+					(size 1.27 1.27)
+				)
+				(hide yes)
+			)
+		)
+		(property "Description" "USB Power-Only 6P Type-C Receptacle connector"
+			(at 74.93 44.45 0)
+			(effects
+				(font
+					(size 1.27 1.27)
+				)
+				(hide yes)
+			)
+		)
+		(pin "A5"
+		)
+		(pin "B9"
+		)
+		(pin "B5"
+		)
+		(pin "A9"
+		)
+		(pin "A12"
+		)
+		(pin "S1"
+		)
+		(pin "B12"
+		)
+		(instances
+			(project ""
+				(path "/804d8951-ccf0-42ec-be9a-378a7536c3df"
+					(reference "J2")
+					(unit 1)
+				)

Commit message: Add additional details.
Parts:
- removed J1: USB_C_Receptacle, symbol Connector:USB_C_Receptacle
- removed J2: USB_C_Receptacle_PowerOnly_6P, symbol Connector:USB_C_Receptacle_PowerOnly_6P
Other:
- note added: "Notes for PCB design: - Stack-up used: SIG, GND, PWR, SIG - Stack-up parameters taken from JLCPCB board stack-up 3313 - JLCPCB calculator used to calculate trace width and spacing for the above stack-up."
- note removed: "Notes for PCB design: - Make four layer board so traces can have controlled impedance with reasonable widths - Check specs for controlled impedance, should be 100R for differential and 50R for single ended - There needs to be ground pore on inner layer for necessary coupling for controlled impedance. - Timing needs to be equal between differential pairs. This can be achieved with length matching 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"
- company: (none) -> Ziad Ibbini
- title: (none) -> RPi HDMi-CSI converter board
Changed lines of the file:
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@@
 	(generator_version "8.0")
 	(paper "A4")
+	(title_block
+		(title "RPi HDMi-CSI converter board")
+		(date "05/24")
+		(rev "v1.1")
+		(company "Ziad Ibbini")
+	)
 	(junction
 		(at 138.43 73.66)
@@
 		)
 	)
-	(text "Notes for PCB design:\n\n- Make four layer board so traces can have controlled \nimpedance with reasonable widths\n- Check specs for controlled impedance, should be 100R for differential\nand 50R for single ended\n- There needs to be ground pore on inner layer for necessary coupling\nfor controlled impedance. \n- Timing needs to be equal between differential pairs. This can be achieved\nwith length matching\n\n\n- Stack-up used: SIG, GND, PWR, SIG\n- Stack-up parameters taken from JLCPCB board stack-up 3313\n- JLCPCB calculator used to calculate trace width and spacing for \nthe above stack-up.\n\n\n"
+	(text "Notes for PCB design:\n- Stack-up used: SIG, GND, PWR, SIG\n- Stack-up parameters taken from JLCPCB board stack-up 3313\n- JLCPCB calculator used to calculate trace width and spacing for \nthe above stack-up.\n\n\n"
 		(exclude_from_sim no)
-		(at 18.288 161.036 0)
+		(at 55.626 148.59 0)
 		(effects
 			(font
@@
 			)
 			(justify right bottom)
-		)
-	)
-	(symbol
-		(lib_id "Connector:USB_C_Receptacle")
-		(at 35.56 59.69 0)
-		(unit 1)
-		(exclude_from_sim no)
-		(in_bom yes)
-		(on_board yes)
-		(dnp no)
-		(fields_autoplaced yes)
-		(property "Reference" "J1"
-			(at 35.56 26.67 0)
-			(effects
-				(font
-					(size 1.27 1.27)
-				)
-			)
-		)
-		(property "Value" "USB_C_Receptacle"
-			(at 35.56 29.21 0)
-			(effects
-				(font
-					(size 1.27 1.27)
-				)
-			)
-		)
-		(property "Footprint" ""
-			(at 39.37 59.69 0)
-			(effects
-				(font
-					(size 1.27 1.27)
-				)
-				(hide yes)
-			)
-		)
-		(property "Datasheet" "https://www.usb.org/sites/default/files/documents/usb_type-c.zip"
-			(at 39.37 59.69 0)
-			(effects
-				(font
-					(size 1.27 1.27)
-				)
-				(hide yes)
-			)
-		)
-		(property "Description" "USB Full-Featured Type-C Receptacle connector"
-			(at 35.56 59.69 0)
-			(effects
-				(font
-					(size 1.27 1.27)
-				)
-				(hide yes)
-			)
-		)
-		(pin "A6"
-		)
-		(pin "B3"
-		)
-		(pin "B9"
-		)
-		(pin "A7"
-		)
-		(pin "B4"
-		)
-		(pin "A1"
-		)
-		(pin "B10"
-		)
-		(pin "A12"
-		)
-		(pin "A8"
-		)
-		(pin "A11"
-		)
-		(pin "S1"
-		)
-		(pin "B12"
-		)
-		(pin "B7"
-		)
-		(pin "A4"
-		)
-		(pin "A5"
-		)
-		(pin "B6"
-		)
-		(pin "B8"
-		)
-		(pin "A2"
-		)
-		(pin "A10"
-		)
-		(pin "A9"
-		)
-		(pin "B5"
-		)
-		(pin "B1"
-		)
-		(pin "B2"
-		)
-		(pin "B11"
-		)
-		(pin "A3"
-		)
-		(instances
-			(project ""
-				(path "/804d8951-ccf0-42ec-be9a-378a7536c3df"
-					(reference "J1")
-					(unit 1)
-				)
-			)
 		)
 	)
@@
 					(unit 1)
 				)
-			)
-		)
-	)
-	(symbol
-		(lib_id "Connector:USB_C_Receptacle_PowerOnly_6P")
-		(at 74.93 44.45 0)
-		(unit 1)
-		(exclude_from_sim no)
-		(in_bom yes)
-		(on_board yes)
-		(dnp no)
-		(fields_autoplaced yes)
-		(property "Reference" "J2"
-			(at 74.93 26.67 0)
-			(effects
-				(font
-					(size 1.27 1.27)
-				)
-			)
-		)
-		(property "Value" "USB_C_Receptacle_PowerOnly_6P"
-			(at 74.93 29.21 0)
-			(effects
-				(font
-					(size 1.27 1.27)
-				)
-			)
-		)
-		(property "Footprint" ""
-			(at 78.74 41.91 0)
-			(effects
-				(font
-					(size 1.27 1.27)
-				)
-				(hide yes)
-			)
-		)
-		(property "Datasheet" "https://www.usb.org/sites/default/files/documents/usb_type-c.zip"
-			(at 74.93 44.45 0)
-			(effects
-				(font
-					(size 1.27 1.27)
-				)
-				(hide yes)
-			)
-		)
-		(property "Description" "USB Power-Only 6P Type-C Receptacle connector"
-			(at 74.93 44.45 0)
-			(effects
-				(font
-					(size 1.27 1.27)
-				)
-				(hide yes)
-			)
-		)
-		(pin "A5"
-		)
-		(pin "B9"
-		)
-		(pin "B5"
-		)
-		(pin "A9"
-		)
-		(pin "A12"
-		)
-		(pin "S1"
-		)
-		(pin "B12"
-		)
-		(instances
-			(project ""
-				(path "/804d8951-ccf0-42ec-be9a-378a7536c3df"
-					(reference "J2")
-					(unit 1)
-				)
